Commit message: update on my current work status

File: ros/src/gazebo-simulation/resource/models/car/car.urdf.xacro (robot description, xacro)
@@ -38,6 +38,6 @@
   <xacro:property name="axle_effort" value="100"/>
   <xacro:property name="axle_velocity" value="100"/>
-  <material name="Green">
-    <color rgba="0 1.0 0 1.0"/>
+  <material name="Red">
+    <color rgba="1.0 0 0 1.0"/>
   </material>
   <!-- general wheel macro without functionality -->
@@ -130,5 +130,5 @@
   </link>
   <gazebo reference="chassis">
-    <material>Gazebo/Green</material>
+    <material>Gazebo/Purple</material>
   </gazebo>
   <joint name="base_link_to_chassis" type="fixed">
@@ -231,5 +231,8 @@
   <xacro:rear_wheel lr_prefix="left" fr_prefix="rear" lr_reflect="${left}" wheel_pos="${rear_wheel_pos}"/>
   <xacro:rear_wheel lr_prefix="right" fr_prefix="rear" lr_reflect="${right}" wheel_pos="${rear_wheel_pos}"/>
-  <xacro:lidar_sensor idx="0" xyz="0.05 0.1 0.018" angle="1.5707963267948966"/>
+  <xacro:lidar_sensor idx="Front_Left" xyz="0.05 0.1 0.018" angle="1.5707963267948966"/>
+  <xacro:lidar_sensor idx="Front_Right" xyz="0.05 -0.1 0.018" angle="-1.5707963267948966"/>
+  <xacro:lidar_sensor idx="Front" xyz="0.15 0 0.018" angle="0"/>
+  <xacro:lidar_sensor idx="Back" xyz="-0.15 0 0.018" angle="3.141592"/>
   <xacro:camera_sensor xyz="-0.07 0 0.185" pitch="-0.1"/>
   <ros2_control name="GazeboSystem" type="system">

Commit message: back to real top down and advance steering

File: ros/src/gazebo-simulation/resource/models/car/car.urdf.xacro (robot description, xacro)
@@ -193,4 +193,45 @@
     </gazebo>
   </xacro:macro>
+  <xacro:macro name="lidar_sensor_lane" params="idx xyz angle">
+    <link name="lidar_link_${idx}">
+      <!--xacro:null_inertial/-->
+    </link>
+    <joint name="lidar_joint_${idx}" type="fixed">
+      <axis xyz="0 0 -1"/>
+      <origin xyz="${xyz}" rpy="0 0 ${angle}"/>
+      <parent link="base_link"/>
+      <child link="lidar_link_${idx}"/>
+    </joint>
+    <gazebo reference="lidar_link_${idx}">
+      <sensor type="ray" name="lidar_sensor_${idx}">
+        <pose>0 0 0 0 0 0</pose>
+        <visualize>true</visualize>
+        <update_rate>5</update_rate>
+        <ray>
+          <scan>
+            <horizontal>
+              <samples>2</samples>
+              <resolution>1</resolution>
+              <min_angle>-0.027</min_angle>
+              <max_angle>0.027</max_angle>
+            </horizontal>
+          </scan>
+          <range>
+            <min>0.10</min>
+            <max>1.5</max>
+            <resolution>0.009</resolution>
+          </range>
+        </ray>
+        <plugin name="scan" filename="libgazebo_ros_ray_sensor.so">
+          <ros>
+            <remapping>~/out:=tof_${idx}</remapping>
+          </ros>
+          <output_type>sensor_msgs/Range</output_type>
+          <frame_name>tof_${idx}</frame_name>
+          <radiation_type>ultrasound</radiation_type>
+        </plugin>
+      </sensor>
+    </gazebo>
+  </xacro:macro>
   <xacro:macro name="camera_sensor" params="xyz pitch">
     <link name="camera_link">
@@ -235,5 +276,6 @@
   <xacro:lidar_sensor idx="Front" xyz="0.15 0 0.018" angle="0"/>
   <xacro:lidar_sensor idx="Back" xyz="-0.15 0 0.018" angle="3.141592"/>
-  <xacro:camera_sensor xyz="-0.07 0 0.185" pitch="-0.1"/>
+  <xacro:lidar_sensor_lane idx="Front2" xyz="0.15 0 0.018" angle="0"/>
+  <xacro:camera_sensor xyz="0.6 0 1" pitch="1.57"/>
   <ros2_control name="GazeboSystem" type="system">
     <hardware>

Commit message: boxes are now being ignored in line image

File: ros/src/gazebo-simulation/resource/models/car/car.urdf.xacro (robot description, xacro)
@@ -39,5 +39,5 @@
   <xacro:property name="axle_velocity" value="100"/>
   <material name="Red">
-    <color rgba="1.0 0 0 1.0"/>
+    <color rgba="1.0 0.7 1.0 1.0"/>
   </material>
   <!-- general wheel macro without functionality -->
@@ -81,4 +81,5 @@
       <kd>1</kd>
       <kp>100000000</kp>
+      <material>Gazebo/Purple</material>
     </gazebo>
   </xacro:macro>

Commit message: overtaker clean-up, parking fixes, velocity_controller initiation and more

File: ros/src/gazebo-simulation/resource/models/car/car.urdf.xacro (robot description, xacro)
@@ -153,4 +153,5 @@
     </sensor>
   </gazebo>
+<!-- Normal ToF Sensor -->
   <xacro:macro name="lidar_sensor" params="idx xyz angle">
     <link name="lidar_link_${idx}">
@@ -194,4 +195,5 @@
     </gazebo>
   </xacro:macro>
+<!-- Modified ToF sensor (for overtaker) -->
   <xacro:macro name="lidar_sensor_lane" params="idx xyz angle">
     <link name="lidar_link_${idx}">
@@ -235,4 +237,52 @@
     </gazebo>
   </xacro:macro>
+<!-- Laser Sensor (for velocity control) -->
+  <xacro:macro name="lidar_sensor_laser" params="idx xyz angle">
+    <link name="lidar_link_${idx}">
+      <!--xacro:null_inertial/-->
+    </link>
+    <joint name="lidar_joint_${idx}" type="fixed">
+      <axis xyz="0 0 -1"/>
+      <origin xyz="${xyz}" rpy="0 0 ${angle}"/>
+      <parent link="base_link"/>
+      <child link="lidar_link_${idx}"/>
+    </joint>
+    <gazebo reference="lidar_link_${idx}">
+      <sensor type="ray" name="lidar_sensor_${idx}">
+        <pose>0 0 0 0 0 0</pose>
+        <always_on>true</always_on>
+        <visualize>true</visualize>
+        <update_rate>5</update_rate>
+        <ray>
+          <scan>
+            <horizontal>
+              <samples>360</samples>
+              <resolution>1.00000</resolution>
+              <min_angle>0.000000</min_angle>
+              <max_angle>6.280000</max_angle>
+            </horizontal>
+          </scan>
+          <range>
+            <min>0.120000</min>
+            <max>3.5</max>
+            <resolution>0.015000</resolution>
+          </range>
+          <noise>
+            <type>gaussian</type>
+            <mean>0.0</mean>
+            <stddev>0.01</stddev>
+          </noise>
+        </ray>
+        <plugin name="scan" filename="libgazebo_ros_ray_sensor.so">
+          <ros>
+            <remapping>~/out:=tof_${idx}</remapping>
+          </ros>
+          <output_type>sensor_msgs/LaserScan</output_type>
+          <frame_name>tof_${idx}</frame_name>
+        </plugin>
+      </sensor>
+    </gazebo>
+  </xacro:macro>
+<!-- Camera sensor -->
   <xacro:macro name="camera_sensor" params="xyz pitch">
     <link name="camera_link">
@@ -279,4 +329,5 @@
   <xacro:lidar_sensor_lane idx="Front2" xyz="0.15 0 0.018" angle="0"/>
   <xacro:camera_sensor xyz="0.6 0 1" pitch="1.57"/>
+  <xacro:lidar_sensor_laser idx="Top" xyz ="0 0 0.08" angle="0"/>
   <ros2_control name="GazeboSystem" type="system">
     <hardware>
